File: poe4pi.kicad_pcb (KiCad board)
At the start: 2 copper layers, 65.2 x 56.2 mm, 0 parts

Commit message: feat: header placement
Parts:
- added C1: 47 uf, Capacitor_SMD:C_1210_3225Metric, F.Cu at (122.6, 62.9)
- added C15: 100nF 100V, Capacitor_SMD:C_0402_1005Metric, F.Cu at (123.5, 92.0)
- added C2: 47 uf, Capacitor_SMD:C_1210_3225Metric, F.Cu at (122.6, 67.2)
- added C3: 47 uf, Capacitor_SMD:C_1210_3225Metric, F.Cu at (122.6, 71.4)
- added C4: 47 uf, Capacitor_SMD:C_1210_3225Metric, F.Cu at (122.6, 75.7)
- added C5: 47 uf, Capacitor_SMD:C_1210_3225Metric, F.Cu at (122.6, 79.9)
- added C6: 47 uf, Capacitor_SMD:C_1210_3225Metric, F.Cu at (122.6, 84.2)
- added D1: DF01S, Diode_SMD:Diode_Bridge_OnSemi_SDIP-4L, F.Cu at (26.2, 104.7)
- added D2: DF01S, Diode_SMD:Diode_Bridge_OnSemi_SDIP-4L, F.Cu at (38.9, 102.7)
- added D4: SMAJ58A, Diode_SMD:D_SMA, F.Cu at (93.7, 102.1)
- added H1: MountingHole, MountingHole:MountingHole_2.5mm, F.Cu at (31.5, 36.5)
- added H2: MountingHole, MountingHole:MountingHole_2.5mm, F.Cu at (31.5, 85.5)
- added H3: MountingHole, MountingHole:MountingHole_2.5mm, F.Cu at (89.5, 36.5)
- added H4: MountingHole, MountingHole:MountingHole_2.5mm, F.Cu at (89.5, 85.5)
- added J1: Conn_02x02_Odd_Even, Connector_PinSocket_2.54mm:PinSocket_2x02_P2.54mm_Vertical, F.Cu at (87.7, 96.9)
- added J2: Conn_02x02_Odd_Even, Connector_PinSocket_2.54mm:PinSocket_2x02_P2.54mm_Vertical, F.Cu at (87.7, 101.5)
- added J3: Conn_02x20_Odd_Even, Connector_PinHeader_2.54mm:PinHeader_2x20_P2.54mm_Vertical, F.Cu at (36.5, 37.8)
- added LSI-U1: lsi-powermodule-7, lsi:lsi-powermodule-7, F.Cu at (112.2, 103.9)
- added LSI-U2: lsi-powermodule-7, lsi:lsi-powermodule-7, F.Cu at (51.2, 97.4)
- added R1: 0, Resistor_SMD:R_0402_1005Metric, F.Cu at (83.1, 96.3)
- added R12: 0, Resistor_SMD:R_0402_1005Metric, F.Cu at (83.1, 98.3)
- added R2: 20m, Resistor_SMD:R_01005_0402Metric, F.Cu at (120.9, 91.8)
- added R22: 24.9K, Resistor_SMD:R_0402_1005Metric, F.Cu at (83.1, 100.2)
- added R23: 180K, Resistor_SMD:R_0402_1005Metric, F.Cu at (83.1, 102.2)
- added R24: 4.42K, Resistor_SMD:R_0402_1005Metric, F.Cu at (83.1, 104.2)
- added R3: 20m, Resistor_SMD:R_01005_0402Metric, F.Cu at (120.9, 93.5)
- added R4: 100m, Resistor_SMD:R_1210_3225Metric, F.Cu at (128.6, 62.9)
- added R5: 100m, Resistor_SMD:R_1210_3225Metric, F.Cu at (128.6, 67.1)
- added U1: LTC4413EDD-2-PBF, footprints:DFN-10_DD_LIT, F.Cu at (122.6, 88.7)
- added U3: TPS2375-1, Package_SO:TSSOP-8_4.4x3mm_P0.65mm, F.Cu at (94.0, 97.6)
Other:
- board size 65.2 x 56.2 mm -> 65 x 56 mm

Commit message: feat: initial layout
Parts:
- moved R4 97.7 mm to (33.2, 41.8), turned to 180 degrees
- moved R3 95.8 mm to (31.8, 58.5), turned to -90 degrees
- moved R5 95.4 mm to (33.2, 66.0), turned to 180 degrees
- moved R2 94.7 mm to (31.8, 60.0), turned to 90 degrees
- moved U1 92.9 mm to (34.6, 59.2), turned to 180 degrees
- moved C3 91.4 mm to (33.2, 52.2)
- moved C2 91.2 mm to (33.2, 48.8)
- moved C1 91.1 mm to (33.2, 45.2)
- moved C6 89.7 mm to (33.2, 76.5)
- moved C5 89.6 mm to (33.2, 73.0)
- moved C4 89.6 mm to (33.2, 69.5)
- moved D1 70.7 mm to (84.0, 64.0)
- moved D2 65.6 mm to (84.0, 55.0)
- moved C15 58.1 mm to (73.8, 62.0), turned to 90 degrees
- moved LSI-U1 56.0 mm to (64.2, 75.0), turned to 180 degrees
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Connections:
- LSI-U1 pad 1: unconnected-(LSI-U1-GND-Pad1) -> GND
- LSI-U1 pad 2: unconnected-(LSI-U1-VPP_IN-Pad2) -> POE_V+
- LSI-U2 pad 1: unconnected-(LSI-U2-GND-Pad1) -> GND
- LSI-U2 pad 2: unconnected-(LSI-U2-VPP_IN-Pad2) -> POE_V+
Routing:
- net POE_V+: track 0.00 -> 73.2 mm, vias 0 -> 4
- net POE_PAIR_2-: track 0.00 -> 43.9 mm, vias 0 -> 1
- net POE_PAIR_1-: track 0.00 -> 42.1 mm, vias 0 -> 1
- net POE_PAIR_2+: track 0.00 -> 41.6 mm
- net POE_PAIR_1+: track 0.00 -> 41.5 mm, vias 0 -> 1
- net Net-(U3-PG): track 0.00 -> 29.0 mm, vias 0 -> 2
- net POE_V-: track 0.00 -> 24.1 mm, vias 0 -> 2
- net Net-(LSI-U1-VPP_OUT): track 0.00 -> 22.0 mm
- net Net-(LSI-U2-VPP_OUT): track 0.00 -> 22.0 mm
- net +5V: track 0.00 -> 15.8 mm, vias 0 -> 5
- net GND: track 0.00 -> 11.4 mm, vias 0 -> 4
- net Net-(LSI-U2-S2): track 0.00 -> 9.84 mm
- net Net-(LSI-U1-S2): track 0.00 -> 9.84 mm
- net Net-(C4-Pad2): track 0.00 -> 3.51 mm
- net Net-(C1-Pad2): track 0.00 -> 3.51 mm
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- added copper zone on In2.Cu, net +5V
- added copper zone on B.Cu, net GND
- added copper zone on F.Cu, net GND
- added copper zone on In1.Cu, net GND
Other:
- outline, holes or cut-outs redrawn
- copper layers 2 -> 4

Commit message: feat: v0.1
Parts:
- added G***: LOGO, logos:heimonen solutions small, F.Cu at (60.5, 83.5)
Routing:
- net POE_V+: track 73.2 -> 91.5 mm, vias 4 -> 12
- net +5V: track 15.8 -> 18.9 mm, vias 5 -> 24
- net GND: vias 4 -> 7
Other:
- board text added: "POE4PI v0.1"
