File: poe4pi.kicad_sch (KiCad schematic)
At the start: 24 parts, among them J1 Conn_02x02_Odd_Even, J2 Conn_02x02_Odd_Even, J3 Conn_02x20_Odd_Even, U1 LTC4413EDD-2-PBF, U3 TPS2375-1

Commit message: feat: header placement
Parts:
- added H1, H2, H3, H4: MountingHole, MountingHole:MountingHole_2.5mm, symbol Mechanical:MountingHole
- added R4, R5: 100m, Resistor_SMD:R_1210_3225Metric, symbol Device:R
- D1, D2: footprint Diode_THT:Diode_Bridge_Round_D9.8mm -> Diode_SMD:Diode_Bridge_OnSemi_SDIP-4L
- J1, J2: footprint Connector_PinSocket_1.27mm:PinSocket_2x02_P1.27mm_Vertical -> Connector_PinSocket_2.54mm:PinSocket_2x02_P2.54mm_Vertical
- J3: footprint (none) -> Connector_PinHeader_2.54mm:PinHeader_2x20_P2.54mm_Vertical
Connections:
- net GND: now also R4.2, R5.2; no longer C1.2, C4.2
- new net: C4.2, R5.1
- new net: C1.2, R4.1
Other:
- moved on the sheet: D1, D2

Commit message: feat: initial layout
Connections:
- net GND: now also LSI-U1.1 (GND), LSI-U2.1 (GND)
- net POE_V+: now also LSI-U1.2 (VPP_IN), LSI-U2.2 (VPP_IN)
Changed lines of the file:
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@@
 	)
 	(junction
+		(at 95.25 30.48)
+		(diameter 0)
+		(color 0 0 0 0)
+	)
+	(junction
 		(at 40.64 50.8)
 		(diameter 0)
@@
 	)
 	(junction
+		(at 83.82 30.48)
+		(diameter 0)
+		(color 0 0 0 0)
+	)
+	(junction
 		(at 66.04 50.8)
 		(diameter 0)
@@
 	(wire
 		(pts
+			(xy 100.33 52.07) (xy 113.03 52.07)
+		)
+		(stroke
+			(width 0)
+			(type default)
+		)
+	)
+	(wire
+		(pts
 			(xy 73.66 43.18) (xy 73.66 45.72)
 		)
@@
 	(wire
 		(pts
+			(xy 100.33 30.48) (xy 95.25 30.48)
+		)
+		(stroke
+			(width 0)
+			(type default)
+		)
+	)
+	(wire
+		(pts
 			(xy 40.64 30.48) (xy 55.88 30.48)
 		)
@@
 	(wire
 		(pts
+			(xy 95.25 25.4) (xy 113.03 25.4)
+		)
+		(stroke
+			(width 0)
+			(type default)
+		)
+	)
+	(wire
+		(pts
 			(xy 40.64 50.8) (xy 55.88 50.8)
 		)
@@
 	(wire
 		(pts
+			(xy 95.25 30.48) (xy 95.25 25.4)
+		)
+		(stroke
+			(width 0)
+			(type default)
+		)
+	)
+	(wire
+		(pts
 			(xy 102.87 38.1) (xy 102.87 59.69)
 		)
@@
 	(wire
 		(pts
+			(xy 100.33 30.48) (xy 100.33 52.07)
+		)
+		(stroke
+			(width 0)
+			(type default)
+		)
+	)
+	(wire
+		(pts
+			(xy 83.82 30.48) (xy 95.25 30.48)
+		)
+		(stroke
+			(width 0)
+			(type default)
+		)
+	)
+	(wire
+		(pts
 			(xy 93.98 38.1) (xy 102.87 38.1)
 		)
@@
 	(symbol
 		(lib_id "power:GND")
+		(at 113.03 27.94 270)
+		(unit 1)
+		(exclude_from_sim no)
+		(in_bom yes)
+		(on_board yes)
+		(dnp no)
+		(fields_autoplaced yes)
+		(property "Reference" "#PWR032"
+			(at 106.68 27.94 0)
+			(effects
+				(font
+					(size 1.27 1.27)
+				)
+				(hide yes)
+			)
+		)
+		(property "Value" "GND"
+			(at 109.22 27.9399 90)
+			(effects
+				(font
+					(size 1.27 1.27)
+				)
+				(justify right)
+			)
+		)
+		(property "Footprint" ""
+			(at 113.03 27.94 0)
+			(effects
+				(font
+					(size 1.27 1.27)
+				)
+				(hide yes)
+			)
+		)
+		(property "Datasheet" ""
+			(at 113.03 27.94 0)
+			(effects
+				(font
+					(size 1.27 1.27)
+				)
+				(hide yes)
+			)
+		)
+		(property "Description" "Power symbol creates a global label with name \"GND\" , ground"
+			(at 113.03 27.94 0)
+			(effects
+				(font
+					(size 1.27 1.27)
+				)
+				(hide yes)
+			)
+		)
+		(pin "1"
+		)
+		(instances
+			(project "poe4pi"
+				(path "/2e751bc8-7420-47df-869b-2f102aa561cb"
+					(reference "#PWR032")
+					(unit 1)
+				)
+			)
+		)
+	)
+	(symbol
+		(lib_id "power:GND")
 		(at 139.7 116.84 180)
 		(unit 1)
@@
 					(unit 1)
 				)
+			)
+		)
+	)
+	(symbol
+		(lib_id "power:GND")
+		(at 113.03 54.61 270)
+		(unit 1)
+		(exclude_from_sim no)
+		(in_bom yes)
+		(on_board yes)
+		(dnp no)
+		(fields_autoplaced yes)
+		(property "Reference" "#PWR031"
+			(at 106.68 54.61 0)
+			(effects
+				(font
+					(size 1.27 1.27)
+				)
+				(hide yes)
+			)
+		)
+		(property "Value" "GND"
+			(at 109.22 54.6099 90)
+			(effects
+				(font
+					(size 1.27 1.27)
+				)
+				(justify right)
+			)
+		)
+		(property "Footprint" ""
+			(at 113.03 54.61 0)
+			(effects
+				(font
+					(size 1.27 1.27)
+				)
+				(hide yes)
+			)
+		)
+		(property "Datasheet" ""
+			(at 113.03 54.61 0)
+			(effects
+				(font
+					(size 1.27 1.27)
+				)
+				(hide yes)
+			)
+		)
+		(property "Description" "Power symbol creates a global label with name \"GND\" , ground"
+			(at 113.03 54.61 0)
+			(effects
+				(font
+					(size 1.27 1.27)
+				)
+				(hide yes)
+			)
+		)
+		(pin "1"
+		)
+		(instances
+			(project "poe4pi"
+				(path "/2e751bc8-7420-47df-869b-2f102aa561cb"
+					(reference "#PWR031")
+					(unit 1)
+				)

Commit message: feat: v0.1
Other:
- moved on the sheet: H1, H2, H3, H4, J3
